File: SuperPower-uC/original/mcu.sch (KiCad schematic (older format))
At the start: 1 part, among them U1 ESP32-WROOM-32

Commit message: annotated correctly
Parts:
- renumbered U1 to U2
Changed lines of the file:
@@
 D-
 $Comp
-L RF_Module:ESP32-WROOM-32 U1
+L RF_Module:ESP32-WROOM-32 U2
 U 1 1 5F7CF431
 P 4700 2350
-F 0 "U1" H 4700 3931 50  0000 C CNN
+F 0 "U2" H 4700 3931 50  0000 C CNN
 F 1 "ESP32-WROOM-32" H 4700 3840 50  0000 C CNN
 F 2 "RF_Module:ESP32-WROOM-32" H 4700 850 50  0001 C CNN
